Commit message: add pineapple model

File: unitree_robots/pineapple/urdf/pineapple.urdf (robot description, URDF)
Before this commit: robot pineapple0916, 10 links, 9 joints
Links:
- removed link L_thigh
- added link L_thgih, mass 0.98; collision mesh filename=../meshes/L_thgih_collision.STL; visual mesh filename=../meshes/L_thgih.STL
- link L_calf: mass 0.50000000 -> 0.567; geometry collision mesh filename=../meshes/L_calf_collision.STL; visual mesh filename=../meshes/L_calf.STL
- link L_hip: mass 0.57300000 -> 0.585; geometry visual mesh filename=../meshes/L_hip.STL
- link L_wheel: mass 0.30500000 -> 0.3; geometry collision cylinder length=0.023 radius=0.075; visual mesh filename=../meshes/L_wheel.STL
- link R_calf: mass 0.50000000 -> 0.567; geometry collision mesh filename=../meshes/R_calf_collision.STL; visual mesh filename=../meshes/R_calf.STL
- link R_hip: mass 0.57300000 -> 0.585; geometry visual mesh filename=../meshes/R_hip.STL
- link R_thigh: mass 0.75000000 -> 0.98; geometry collision mesh filename=../meshes/R_thigh_collision.STL; visual mesh filename=../meshes/R_thigh.STL
- link R_wheel: mass 0.30500000 -> 0.3; geometry collision cylinder length=0.023 radius=0.075; visual mesh filename=../meshes/R_wheel.STL
- link base_link: mass 2.85000000 -> 3.63; geometry collision mesh filename=../meshes/base_link_collision.STL; visual mesh filename=../meshes/base_link.STL
- link cam: mass 0.30000000 -> 0.3; geometry visual mesh filename=../meshes/cam.STL
Joints:
- joint L_calf_joint: limit lower=-3.1416 upper=0.0 effort=33.5 velocity=21.0 -> lower=-3.141 upper=0 effort=23.7 velocity=30.1; origin xyz=0 0.035931787557176 -0.190000001217773 rpy=0 0 0 -> xyz=0 0.04135 -0.165 rpy=0 0 0; parent L_thigh -> L_thgih
- joint L_hip_joint: limit lower=-0.52358 upper=0.17444 effort=23.7 velocity=30.0 -> lower=-0.52358 upper=0.17444 effort=23.7 velocity=30.1; origin xyz=0 0.06125 0 rpy=0 0 0 -> xyz=0 0.061689 0.066 rpy=0 0 0
- joint L_thigh_joint: child L_thigh -> L_thgih; limit lower=0.0 upper=1.571 effort=23.7 velocity=30.0 -> lower=0 upper=1.57 effort=23.7 velocity=30.1; origin xyz=0 0.0129353215081658 0 rpy=0 0 0 -> xyz=0 0.027596 0 rpy=0 0 0
- joint L_wheel_joint: origin xyz=0 0.0421817504179199 -0.190000000000001 rpy=0 0 0 -> xyz=0 0.024414 -0.165 rpy=0 0 0; type continuous -> revolute
- joint R_calf_joint: limit lower=-3.1416 upper=0.0 effort=33.5 velocity=21.0 -> lower=-3.141 upper=0 effort=23.7 velocity=30.1; origin xyz=0 -0.0359317875571787 -0.190000001217773 rpy=0 0 0 -> xyz=0 -0.04135 -0.165 rpy=0 0 0
- joint R_hip_joint: limit lower=-0.17444 upper=0.52358 effort=23.7 velocity=30.0 -> lower=-0.17444 upper=0.52358 effort=23.7 velocity=30.1; origin xyz=0 -0.0612499999999985 0 rpy=0 0 0 -> xyz=0 -0.061689 0.066 rpy=0 0 0
- joint R_thigh_joint: limit lower=0.0 upper=1.571 effort=23.7 velocity=30.0 -> lower=0 upper=1.57 effort=23.7 velocity=30.1; origin xyz=0 -0.0129353215081659 0 rpy=0 0 0 -> xyz=0 -0.027596 0 rpy=0 0 0
- joint R_wheel_joint: origin xyz=0 -0.0421817504179163 -0.190000000000001 rpy=0 0 0 -> xyz=0 -0.024414 -0.165 rpy=0 0 0; type continuous -> revolute
- joint cam_joint: origin xyz=0.136663127592924 0 0.0595399140665773 rpy=0 0.698131700797732 0 -> xyz=0.136663127592924 0 0.125539913353642 rpy=0 0.698131700797732 0
