Commit message: fix pineapple v1 urdf and mjcf

File: pineapple_robots/pineapple_v1/urdf/pineapple.urdf (robot description, URDF)
Before this commit: robot pineapple, 10 links, 9 joints
Links:
- removed link L_thgih
- removed link cam
- added link L_thigh, mass 0.911; collision box size=0.055 0.019 0.12; collision cylinder length=0.035 radius=0.0515
- added link battery, mass 0.64; visual mesh filename=package://pineapple v1.1/meshes/battery.STL
- link L_calf: geometry collision box size=0.048 0.0236 0.093; visual mesh filename=package://pineapple v1.1/meshes/L_calf.STL
- link L_hip: geometry visual mesh filename=package://pineapple v1.1/meshes/L_hip.STL
- link L_wheel: mass 0.3 -> 0.35; geometry collision cylinder length=0.023 radius=0.07; visual mesh filename=package://pineapple v1.1/meshes/L_wheel.STL
- link R_calf: geometry collision box size=0.048 0.0236 0.093; visual mesh filename=package://pineapple v1.1/meshes/R_calf.STL
- link R_hip: geometry visual mesh filename=package://pineapple v1.1/meshes/R_hip.STL
- link R_thigh: mass 0.98 -> 0.911; geometry collision box size=0.055 0.019 0.12; collision cylinder length=0.035 radius=0.0515
- link R_wheel: mass 0.3 -> 0.35; geometry collision cylinder length=0.023 radius=0.07; visual mesh filename=package://pineapple v1.1/meshes/R_wheel.STL
- link base_link: mass 3.63 -> 2.99; geometry collision box size=0.05 0.05 0.1; collision box size=0.05 0.05 0.1
Joints:
- removed joint cam_joint
- added joint battery_fix: type fixed, parent base_link, child battery, origin xyz=0 0 0 rpy=0 0 0, axis 0 0 0
- joint L_calf_joint: origin xyz=0 0.04135 -0.165 rpy=0 0 0 -> xyz=0 0.0383 -0.165 rpy=0 0 0; parent L_thgih -> L_thigh
- joint L_hip_joint: origin xyz=0 0.061689 0.066 rpy=0 0 0 -> xyz=0.047159 0.06125 0.066001 rpy=0 0 0
- joint L_thigh_joint: child L_thgih -> L_thigh; origin xyz=0 0.027596 0 rpy=0 0 0 -> xyz=-0.05675 0.01995 0 rpy=0 0 0
- joint L_wheel_joint: limit effort=3.69 velocity=60.0 -> effort=3.69 velocity=60; origin xyz=0 0.024414 -0.165 rpy=0 0 0 -> xyz=0 0.02705 -0.165 rpy=0 0 0; type revolute -> continuous
- joint R_calf_joint: origin xyz=0 -0.04135 -0.165 rpy=0 0 0 -> xyz=0 -0.0383 -0.165 rpy=0 0 0
- joint R_hip_joint: origin xyz=0 -0.061689 0.066 rpy=0 0 0 -> xyz=0.047159 -0.06125 0.066001 rpy=0 0 0
- joint R_thigh_joint: origin xyz=0 -0.027596 0 rpy=0 0 0 -> xyz=-0.05675 -0.01995 0 rpy=0 0 0
- joint R_wheel_joint: limit effort=3.69 velocity=60.0 -> effort=3.69 velocity=60; origin xyz=0 -0.024414 -0.165 rpy=0 0 0 -> xyz=0 -0.02705 -0.165 rpy=0 0 0; type revolute -> continuous
