Commit message: merge v2 with v2_arm

File: pineapple_robots/pineapple_v2_arm/urdf/pineapple_v2_arm.urdf (robot description, URDF)
Before this commit: robot pineapple_v2_arm, 18 links, 17 joints
Links:
- removed link calf_L_link
- removed link calf_R_link
- removed link hip_L_link
- removed link hip_R_link
- removed link thigh_L_link
- removed link thigh_R_link
- removed link wheel_L_link
- removed link wheel_R_link
- added link L_calf, mass 0.353; collision box size=0.052 0.021 0.122; collision cylinder length=0.021 radius=0.026
- added link L_hip, mass 0.894; visual mesh filename=../meshes/L_hip.STL
- added link L_thigh, mass 0.434; collision box size=0.056 0.028 0.11; collision cylinder length=0.028 radius=0.028
- added link L_wheel, mass 0.405; collision cylinder length=0.007 radius=0.077; visual mesh filename=../meshes/L_wheel.STL
- added link R_calf, mass 0.353; collision box size=0.052 0.021 0.122; collision cylinder length=0.021 radius=0.026
- added link R_hip, mass 0.894; visual mesh filename=../meshes/R_hip.STL
- added link R_thigh, mass 0.434; collision box size=0.056 0.028 0.11; collision cylinder length=0.028 radius=0.028
- added link R_wheel, mass 0.405; collision cylinder length=0.007 radius=0.077; visual mesh filename=../meshes/R_wheel.STL
- added link arm_base, mass 0.375; visual mesh filename=../meshes/arm_base.STL
- added link battery, mass 0.76; visual mesh filename=../meshes/battery.STL
- added link camera, mass 0.3; visual mesh filename=../meshes/camera.STL
- added link hip_motor_L, mass 0.55; visual mesh filename=../meshes/hip_motor_L.STL
- added link hip_motor_R, mass 0.55; visual mesh filename=../meshes/hip_motor_R.STL
- added link knee_motor_L, mass 0.93; visual mesh filename=../meshes/knee_motor_L.STL
- added link knee_motor_R, mass 0.93; visual mesh filename=../meshes/knee_motor_R.STL
- added link wheel_motor_L, mass 0.335; visual mesh filename=../meshes/wheel_motor_L.STL
- added link wheel_motor_R, mass 0.335; visual mesh filename=../meshes/wheel_motor_R.STL
- link base_link: mass 3.10800000 -> 1.673
Joints:
- added joint Knee_motor_R_fix: type fixed, parent R_thigh, child knee_motor_R, origin xyz=0 0 0 rpy=0 0 0, axis 0 0 0
- added joint arm_base_fix: type fixed, parent base_link, child arm_base, origin xyz=0 0 0 rpy=0 0 0, axis 0 0 0
- added joint battery_fix: type fixed, parent base_link, child battery, origin xyz=0 0 0 rpy=0 0 0, axis 0 0 0
- added joint camera_fix: type fixed, parent base_link, child camera, origin xyz=0 0 0 rpy=0 0 0, axis 0 0 0
- added joint hip_motor_L_fix: type fixed, parent base_link, child hip_motor_L, origin xyz=0 0 0 rpy=0 0 0, axis 0 0 0
- added joint hip_motor_R_fix: type fixed, parent base_link, child hip_motor_R, origin xyz=0 0 0 rpy=0 0 0, axis 0 0 0
- added joint knee_motor_L_fix: type fixed, parent L_thigh, child knee_motor_L, origin xyz=0 0 0 rpy=0 0 0, axis 0 0 0
- added joint wheel_motor_L_fix: type fixed, parent L_calf, child wheel_motor_L, origin xyz=0 0 0 rpy=0 0 0, axis 0 0 0
- added joint wheel_motor_R_fix: type fixed, parent R_calf, child wheel_motor_R, origin xyz=0 0 0 rpy=0 0 0, axis 0 0 0
- joint L_calf_joint: child calf_L_link -> L_calf; limit (none) -> lower=-3.314 upper=0.174 effort=40.0 velocity=16.76; parent thigh_L_link -> L_thigh
- joint L_hip_joint: child hip_L_link -> L_hip
- joint L_thigh_joint: child thigh_L_link -> L_thigh; parent hip_L_link -> L_hip
- joint L_wheel_joint: child wheel_L_link -> L_wheel; origin xyz=0 0.0355 -0.189999999999999 rpy=0 0 0 -> xyz=0 0.0355 -0.19 rpy=0 0 0; parent calf_L_link -> L_calf
- joint R_calf_joint: child calf_R_link -> R_calf; limit (none) -> lower=-3.314 upper=0.174 effort=40.0 velocity=16.76; parent thigh_R_link -> R_thigh
- joint R_hip_joint: child hip_R_link -> R_hip
- joint R_thigh_joint: child thigh_R_link -> R_thigh; parent hip_R_link -> R_hip
- joint R_wheel_joint: child wheel_R_link -> R_wheel; parent calf_R_link -> R_calf
- joint arm_base_joint: limit lower=-6.283185307179586 upper=6.283185307179586 effort=10.0 velocity=10.0 -> lower=-3.141592653589793 upper=3.141592653589793 effort=10.0 velocity=10.0
- joint arm_link1_joint: limit lower=-6.283185307179586 upper=6.283185307179586 effort=10.0 velocity=10.0 -> lower=0.0 upper=3.141592653589793 effort=10.0 velocity=10.0
- joint arm_link2_joint: limit lower=-6.283185307179586 upper=6.283185307179586 effort=10.0 velocity=10.0 -> lower=-3.141592653589793 upper=0.0 effort=10.0 velocity=10.0
- joint arm_link3_joint: limit lower=-6.283185307179586 upper=6.283185307179586 effort=10.0 velocity=10.0 -> lower=-3.0 upper=1.0 effort=10.0 velocity=10.0
- joint arm_link4_joint: limit lower=-6.283185307179586 upper=6.283185307179586 effort=10.0 velocity=10.0 -> lower=-1.8 upper=2.1 effort=10.0 velocity=10.0
- joint arm_link5_joint: limit lower=-6.283185307179586 upper=6.283185307179586 effort=10.0 velocity=10.0 -> lower=-1.47 upper=1.47 effort=10.0 velocity=10.0
- joint arm_link6_joint: limit lower=-6.283185307179586 upper=6.283185307179586 effort=10.0 velocity=10.0 -> lower=-3.141592653589793 upper=3.141592653589793 effort=10.0 velocity=10.0
