Commit message: fix pineapple_v2_arm

File: pineapple_robots/pineapple_v2_arm/urdf/pineapple_v2_arm.urdf (robot description, URDF)
Before this commit: robot pineappleV2, 27 links, 26 joints
Links:
- removed link arm_base_link
- removed link arm_gripper_link1
- removed link arm_gripper_link2
- removed link arm_link1
- removed link arm_link2
- removed link arm_link3
- removed link arm_link4
- removed link arm_link5
- removed link arm_link6
- added link 5dof, mass 0.54504586; collision box size=0.065 0.065 0.06; visual mesh filename=../meshes/5dof.dae scale=1 1 1
- added link 6dof, mass 0.36685284; collision box size=0.06 0.065 0.072; visual mesh filename=../meshes/6dof.dae scale=1 1 1
- added link fore_arm, mass 0.97574223; collision box size=0.26 0.062 0.06; visual mesh filename=../meshes/fore_arm.dae scale=1 1 1
- added link upper_arm, mass 1.25745063; collision box size=0.353 0.07 0.068; visual mesh filename=../meshes/upper_arm.dae scale=1 1 1
- link arm_base: mass 0.375 -> 0.2549039; geometry visual mesh filename=../meshes/arm_base.dae scale=1 1 1
Joints:
- removed joint arm_gripper_left_joint
- removed joint arm_gripper_right_joint
- removed joint arm_link1_joint
- removed joint arm_link2_joint
- removed joint arm_link3_joint
- removed joint arm_link4_joint
- removed joint arm_link5_joint
- removed joint arm_link6_joint
- added joint 5dof_joint: type revolute, parent 5dof, child 6dof, origin xyz=0.08 -0.0328 0.04075 rpy=0 0 0, axis 0 0 1, limit lower=-1.5708 upper=1.5708 effort=0 velocity=0
- added joint arm_joint: type revolute, parent base_link, child arm_base, origin xyz=0.00095065 -0.00034599 0.12 rpy=0 0 0, axis 0 0 1, limit lower=-1.5708 upper=1.5708 effort=0 velocity=0
- added joint fore_arm_joint: type revolute, parent fore_arm, child 5dof, origin xyz=0.2698 -0.00295 0.075 rpy=0 0 0, axis 0 1 0, limit lower=-1.5708 upper=1.7453 effort=0 velocity=0
- added joint upper_arm_joint: type revolute, parent upper_arm, child fore_arm, origin xyz=-0.3 0.07082 0 rpy=0 0 0, axis 0 1 0, limit lower=-3.1416 upper=0 effort=0 velocity=0
- joint arm_base_joint: axis 0 0 1 -> 0 1 0; child arm_base_link -> upper_arm; limit lower=-3.141592653589793 upper=3.141592653589793 effort=10.0 velocity=10.0 -> lower=0 upper=3.1416 effort=0 velocity=0; origin xyz=0.0311680686284274 -0.00134995018468019 0.148500000000001 rpy=0 0 0 -> xyz=0.0392 -0.0355 0.052 rpy=0 0 0; parent base_link -> arm_base

Commit message: fix pineapple_v2_arm urdf

File: pineapple_robots/pineapple_v2_arm/urdf/pineapple_v2_arm.urdf (robot description, URDF)
Before this commit: robot pineappleV2, 22 links, 22 joints
Links:
- added link gripper_case_link, mass 0.40000000; collision box size=0.05 0.071 0.07; visual mesh filename=package://arm_v3_description/meshes/gripper_case_link.STL
- added link gripper_left_link, mass 0.10000000; collision box size=0.149 0.04 0.0376; visual mesh filename=package://arm_v3_description/meshes/gripper_left_link.STL
- added link gripper_right_link, mass 0.10000000; collision box size=0.149 0.04 0.0376; visual mesh filename=package://arm_v3_description/meshes/gripper_right_link.STL
Joints:
- added joint gripper_case_joint: type revolute, parent 6dof, child gripper_case_link, origin xyz=0.0289999999999858 0 -0.0407499999999717 rpy=0 0 0, axis 1 0 0, limit lower=-1.57 upper=1.57 effort=10 velocity=30
- added joint gripper_left_joint: type prismatic, parent gripper_case_link, child gripper_left_link, origin xyz=0.0743999852684834 0.0602750061962686 -0.000100006520500351 rpy=0 0 0, axis 0 -1 0, limit lower=0 upper=0.04 effort=1 velocity=0.01
- added joint gripper_right_joint: type prismatic, parent gripper_case_link, child gripper_right_link, origin xyz=0.074399994923587 -0.0602749896221725 -0.00010000652049913 rpy=0 0 0, axis 0 -1 0, limit lower=-0.04 upper=0 effort=1 velocity=0.01
