Commit message: update pineapple v2

File: pineapple_robots/pineapple_v2/urdf/pineappleV2.urdf (robot description, URDF)
Before this commit: robot pineappleV2, 18 links, 17 joints
Links:
- link L_wheel: geometry collision cylinder length=0.023 radius=0.077; visual mesh filename=../meshes/L_wheel.STL
- link R_wheel: geometry collision cylinder length=0.023 radius=0.077; visual mesh filename=../meshes/R_wheel.STL
Joints:
- joint L_calf_joint: limit lower=-1.745 upper=1.745 effort=40.0 velocity=10.472 -> lower=-3.314 upper=0.174 effort=40.0 velocity=16.76
- joint L_hip_joint: limit lower=-0.698 upper=0.698 effort=20.0 velocity=12.566 -> lower=-0.698 upper=0.698 effort=20.0 velocity=20.94
- joint L_thigh_joint: limit lower=-0.349 upper=1.919 effort=20.0 velocity=12.566 -> lower=-0.349 upper=1.919 effort=20.0 velocity=20.94
- joint L_wheel_joint: limit effort=11.0 velocity=15.708 -> effort=11.0 velocity=25.13
- joint R_calf_joint: limit lower=-1.745 upper=1.745 effort=40.0 velocity=10.472 -> lower=-3.314 upper=0.174 effort=40.0 velocity=16.76
- joint R_hip_joint: limit lower=-0.698 upper=0.698 effort=20.0 velocity=12.566 -> lower=-0.698 upper=0.698 effort=20.0 velocity=20.94
- joint R_thigh_joint: limit lower=-0.349 upper=1.919 effort=20.0 velocity=12.566 -> lower=-0.349 upper=1.919 effort=20.0 velocity=20.94
- joint R_wheel_joint: limit effort=11.0 velocity=15.708 -> effort=11.0 velocity=25.13

Commit message: update v2 wheels collision

File: pineapple_robots/pineapple_v2/urdf/pineappleV2.urdf (robot description, URDF)
Before this commit: robot pineappleV2, 18 links, 17 joints
Links:
- link L_wheel: geometry collision cylinder length=0.007 radius=0.077; visual mesh filename=../meshes/L_wheel.STL
- link R_wheel: geometry collision cylinder length=0.007 radius=0.077; visual mesh filename=../meshes/R_wheel.STL
